File: daw00/analog_input/analog_input.kicad_sch (KiCad schematic)
At the start: 14 parts, among them J1 Conn_01x03_Male, J2 Conn_01x06_Male, U1 PCM1808

Commit message: Добавил надписи
Parts:
- J1: footprint w_conn_av:jack_3.5_pj313d-smt -> 00-mylib:PJ313
Connections:
- net at J1.2 (Pin_2): now also C6.1; no longer C7.2
- net at J1.3 (Pin_3): now also C7.2; no longer C6.1
Other:
- moved on the sheet: J1
