File: daw00/analog_input/analog_input.kicad_pcb (KiCad board)
At the start: 2 copper layers, 25.4 x 31.8 mm, 15 parts, among them J1 Conn_01x03_Male, J2 Conn_01x06_Male, U1 PCM1808

Commit message: Добавил надписи
Parts:
- added REF**: MountingHole_3.2mm_M3, MountingHole:MountingHole_3.2mm_M3, F.Cu at (23.0, 36.9)
- J1: footprint w_conn_av:jack_3.5_pj313d-smt -> 00-mylib:PJ313
- moved C2 133.7 mm to (6.73, 21.5)
- moved C3 133.7 mm to (8.76, 21.5)
- moved C4 133.7 mm to (7.23, 8.98)
- moved C5 133.7 mm to (8.76, 8.98)
- moved C7 133.7 mm to (17.1, 10.3)
- moved J2 133.7 mm to (9.01, 36.9)
- moved R1 133.7 mm to (5.20, 8.92)
- moved RV1 133.7 mm to (22.0, 19.9)
- moved RV2 133.7 mm to (22.0, 12.5)
- moved U1 133.7 mm to (9.01, 15.3)
- moved C1 133.7 mm to (4.69, 18.1)
- moved C6 133.7 mm to (16.9, 17.4)
- moved R2 133.7 mm to (10.8, 8.92)
- moved REF** 133.7 mm to (23.0, 2.63)
- moved J1 132.6 mm to (20.6, 26.6), turned to 180 degrees
Connections:
- C6 pad 1: Net-(J1-Pin_3) -> Net-(J1-Pin_2)
- C7 pad 2: Net-(J1-Pin_2) -> Net-(J1-Pin_3)
- J2 pad 10: GND -> unconnected-(J2-Pin_10-Pad10)
- J2 pad 4: GND -> unconnected-(J2-Pin_4-Pad4)
- J2 pad 6: GND -> unconnected-(J2-Pin_6-Pad6)
- J2 pad 8: GND -> unconnected-(J2-Pin_8-Pad8)
Routing:
- net Net-(J1-Pin_3): track 11.9 -> 22.2 mm
- net Net-(J1-Pin_2): track 22.8 -> 13.1 mm
Other:
- board size 25.4 x 31.8 mm -> 25.4 x 40.6 mm
