File: daw00/Amplifier.kicad_sch (KiCad schematic)
At the start: 175 parts, among them J1 Power in, J12 Conn_01x06_Male, J13 Conn_01x03_Male, J15 Conn_01x06_Male, J16 +6V, J18 Out, J5 SWD, J6 Out, Q1 2STF2360, U1 LD1086D2T33TR, U10 TPS3828-33DBVT, U11 25AA1024-I/SM, U2 L78L18_SOT89, U3 STM32F030F4Px, U4 TAS6424QDKQRQ1, U5 DLR1160, U6 PCM1808, U7 LP2985-5.0, U8 TAS6424QDKQRQ1, U9 ADAU1466WBCPZ300, X1 SG-8002CA 24.5760M-PCBL3

Commit message: Чтоб не потерялось
Parts:
- removed C1, C48: CAP_10u0_25V_X5R_0805, Capacitor_SMD:C_0805_2012Metric, symbol AMPP_1466_V0-rescue:C-Device
- removed C101, C52, C59, C6: CAP_100n_50V_X7R_0603, Capacitor_SMD:C_0603_1608Metric, symbol AMPP_1466_V0-rescue:C-Device
- removed C16: 2n2, Capacitor_SMD:C_0603_1608Metric, symbol AMPP_1466_V0-rescue:C_micro-my
- removed C2, C4: 0,33uF, Capacitor_SMD:C_0603_1608Metric, symbol AMPP_1466_V0-rescue:C-my
- removed C3, C49, C50, C57, C58: 2.2uF, Capacitor_SMD:C_0805_2012Metric, symbol AMPP_1466_V0-rescue:C-Device
- removed C5: CAP_100n_50V_X7R_0603, Capacitor_SMD:C_0603_1608Metric, symbol RDC4-0027v1-rescue:CAP_100n_50V_X7R_0805-rk-infinitas-rescue-SigmaDSP-ADAU1452-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
- removed C51: CAP_150p_50V_C0G_0603, Capacitor_SMD:C_0603_1608Metric, symbol AMPP_1466_V0-rescue:C-Device
- removed C53: CAP_5n6_50V_X7R_0603, Capacitor_SMD:C_0603_1608Metric, symbol AMPP_1466_V0-rescue:C-Device
- removed C54: CAP_10n_50V_X7R_0603, Capacitor_SMD:C_0603_1608Metric, symbol AMPP_1466_V0-rescue:C-Device
- removed C55, C56: 2n2, Capacitor_SMD:C_0603_1608Metric, symbol AMPP_1466_V0-rescue:C-Device
- removed C60, C62, C9: 100n, Capacitor_SMD:C_0603_1608Metric, symbol AMPP_1466_V0-rescue:C-Device
- removed C61: 10n, Capacitor_SMD:C_0603_1608Metric, symbol AMPP_1466_V0-rescue:C-Device
- removed C63: 10,0uF, Capacitor_SMD:C_0805_2012Metric, symbol AMPP_1466_V0-rescue:C-Device
- removed C7, C8: 100n, Capacitor_SMD:C_0603_1608Metric, symbol AMPP_1466_V0-rescue:C-my
- removed HL5, HL6: LED_SMD_0603_BLUE, LED_SMD:LED_0603_1608Metric_Pad1.05x0.95mm_HandSolder, symbol AMPP_1466_V0-rescue:LED-Device
- removed J1: Power in, my:DG16S-B-02P-13-00A(H), symbol AMPP_1466_V0-rescue:Screw_Terminal_01x02-Connector
- removed J13: Conn_01x03_Male, w_conn_av:jack_3.5_pj313d-smt, symbol AMPP_1466_V0-rescue:Conn_01x03-Connector_Generic
- removed J16: +6V, TerminalBlock_Phoenix:TerminalBlock_Phoenix_MKDS-1,5-2-5.08_1x02_P5.08mm_Horizontal, symbol AMPP_1466_V0-rescue:Screw_Terminal_01x02-Connector
- removed J5: SWD, Connector_JST:JST_XH_B4B-XH-A_1x04_P2.50mm_Vertical, symbol AMPP_1466_V0-rescue:Conn_01x04-Connector_Generic
- removed L17: LQH2MCN470K02, Inductor_SMD:L_Murata_LQH2MCNxxxx02_2.0x1.6mm, symbol AMPP_1466_V0-rescue:L_Small-my
- removed Q1: 2STF2360, Package_TO_SOT_SMD:SOT-89-3, symbol AMPP_1466_V0-rescue:Q_PNP_BCE-Device
- removed R1, R23, R24: 10K, Resistor_SMD:R_0603_1608Metric, symbol AMPP_1466_V0-rescue:R_Small-my
- removed R10, R9: 470, Resistor_SMD:R_0603_1608Metric, symbol AMPP_1466_V0-rescue:R-Device
- removed R11, R12, R13, R14, R15, R17, R19: RES_10K0_1%_0.125W_Thick_0603, Resistor_SMD:R_0603_1608Metric, symbol AMPP_1466_V0-rescue:R-Device
- removed R16, R18: RES_51R0_1%_0.125W_Thick_0603, Resistor_SMD:R_0603_1608Metric, symbol AMPP_1466_V0-rescue:R-Device
- removed R6: 47K, Resistor_SMD:R_0603_1608Metric, symbol AMPP_1466_V0-rescue:R_micro-my
- removed R7: RES_4K7_1%_0.125W_Thick_0603, Resistor_SMD:R_0603_1608Metric, symbol AMPP_1466_V0-rescue:R-Device
- removed R8: RES_1K0_1%_0.125W_Thick_0603, Resistor_SMD:R_0603_1608Metric, symbol AMPP_1466_V0-rescue:R-Device
- removed TP1: Reset, TestPoint:TestPoint_Pad_D1.5mm, symbol AMPP_1466_V0-rescue:TestPoint-Connector
- removed U1: LD1086D2T33TR, Package_TO_SOT_SMD:TO-263-2, symbol AMPP_1466_V0-rescue:LD1086D2T33TR-Regulator_Linear
- removed U10: TPS3828-33DBVT, Package_TO_SOT_SMD:SOT-23-5, symbol AMPP_1466_V0-rescue:TPS3828-my
- removed U11: 25AA1024-I/SM, Package_SO:SOIC-8_3.9x4.9mm_P1.27mm, symbol RDC4-0027v1-rescue:IC_25AA1024-rk-infinitas-rescue-SigmaDSP-ADAU1452-rescue-Sig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
- removed U2: L78L18_SOT89, Package_TO_SOT_SMD:SOT-89-3, symbol AMPP_1466_V0-rescue:L78L18_SOT89-Regulator_Linear
- removed U3: STM32F030F4Px, Package_SO:TSSOP-20_4.4x6.5mm_P0.65mm, symbol AMPP_1466_V0-rescue:STM32F030F4Px-MCU_ST_STM32F0
- removed U5: DLR1160, my:Toslink, symbol AMPP_1466_V0-rescue:toslink-FC684208R-my
- removed U6: PCM1808, Package_SO:TSSOP-14_4.4x5mm_P0.65mm, symbol PCM1808--audio-ADC-rescue:PCM1808-PCM1808-rescue-PCM1808--audio-ADC-rescue
- removed U7: LP2985-5.0, Package_TO_SOT_SMD:SOT-23-5, symbol AMPP_1466_V0-rescue:LP2985-3.3-Regulator_Linear
- removed U9: ADAU1466WBCPZ300, ADAU1466:ADAU1466WBCPZ300, symbol ADAU1466:ADAU1466WBCPZ300
- removed VD1: diode BAS85.115, w_smd_diode:sod80c, symbol AMPP_1466_V0-rescue:D_Small-my
- removed VD2: ES1D, w_smd_diode:do214ac, symbol AMPP_1466_V0-rescue:D-Device
- removed X1: SG-8002CA 24.5760M-PCBL3, Oscillator:Oscillator_SMD_SeikoEpson_SG8002CA-4Pin_7.0x5.0mm, symbol AMPP_1466_V0-rescue:SG-8002CA-Oscillator
- added C1, C6: CAP_10u0_25V_X5R_0805, Capacitor_SMD:C_0805_2012Metric, symbol Device:C
- added C3, C50, C53: CAP_100n_50V_X7R_0603, Capacitor_SMD:C_0603_1608Metric, symbol Device:C
- added C48: CAP_150p_50V_C0G_0603, Capacitor_SMD:C_0603_1608Metric, symbol Device:C
- added C51: CAP_5n6_50V_X7R_0603, Capacitor_SMD:C_0603_1608Metric, symbol Device:C
- added C52: CAP_10n_25V_X7R_0603, Capacitor_SMD:C_0603_1608Metric, symbol Device:C
- added HL5, HL6: LED_SMD_0603_BLUE, LED_SMD:LED_0603_1608Metric_Pad1.05x0.95mm_HandSolder, symbol Device:LED
- added J13: Conn_01x04_Male, Connector_PinHeader_2.54mm:PinHeader_1x04_P2.54mm_Vertical, symbol AMPP_1466_V0-rescue:Conn_01x04_Male-Connector
- added J19, J20: Conn_01x06_Male, Connector_Edge:2x6, symbol Connector_Generic:Conn_02x06_Odd_Even
- added J21, J7: Conn_01x02_Male, Connector_PinHeader_2.54mm:PinHeader_1x02_P2.54mm_Vertical, symbol AMPP_1466_V0-rescue:Conn_01x02_Male-Connector
- added Q1: 2STF2360, Package_TO_SOT_SMD:SOT-89-3, symbol Device:Q_PNP_BCE
- added R10, R11, R12, R13, R15, R17, R9: RES_10K0_1%_0.125W_Thick_0603, Resistor_SMD:R_0603_1608Metric, symbol Device:R
- added R14, R16: RES_51R0_1%_0.125W_Thick_0603, Resistor_SMD:R_0603_1608Metric, symbol Device:R
- added R7: RES_4K3_1%_0.125W_Thick_0603, Resistor_SMD:R_0603_1608Metric, symbol Device:R
- added R8: RES_1K0_1%_0.125W_Thick_0603, Resistor_SMD:R_0603_1608Metric, symbol Device:R
- added U6: ADAU1467WBCPZ300RL, my:LFCSP-88-1EP_10x10mm_P0.5mm_EP6.15x6.15mm, symbol AMPP_1466_V0-rescue:ADAU1467-Analog1467-ADAU
- added U9: 25AA1024-I/SM, Package_SO:SOIC-8_3.9x4.9mm_P1.27mm, symbol RDC4-0027v1-rescue:IC_25AA1024-rk-infinitas-rescue-SigmaDSP-ADAU1452-rescue-Sig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
- added X1: SG-8002CA 24.5760M-PCBL3, Oscillator:Oscillator_SMD_SeikoEpson_SG8002CA-4Pin_7.0x5.0mm, symbol Oscillator:SG-8002CA
- FER1, FER2: MP BLM21AG102SN1D -> (none)
- J12: footprint Connector_JST:JST_XH_B6B-XH-A_1x06_P2.50mm_Vertical -> Connector_Edge:2x6; symbol AMPP_1466_V0-rescue:Conn_01x06-Connector_Generic -> Connector_Generic:Conn_02x06_Odd_Even; Поле4 I2S input 0 -> I2S in/out3
- J15: value Conn_01x06_Male -> Volume; symbol AMPP_1466_V0-rescue:Conn_01x06-Connector_Generic -> Connector_Generic:Conn_01x03
- L1, L10, L11, L12, L13, L14, L15, L16, L2, L3, L4, L5, L6, L7, L8, L9: footprint my:Panasonic_ETQP_5.5x5.0x3.0 -> my:SPM5010-5020
Connections:
- net SDA is gone; now on net SCL: R5.2, U4.21 (SDA), U8.21 (SDA)
- net +3V3: now also J12.11 (Pin_11), J15.3 (Pin_3), C52.1, C53.1, J19.11 (Pin_11), J20.11 (Pin_11), Q1.3 (E), R10.1, R11.1, R12.1, R13.1, R14.1, R15.1, R16.1, R17.1, R8.2, R9.1, U6.2 (IOVDD), U6.22 (IOVDD), U6.37 (IOVDD), U6.46 (IOVDD), U6.68 (IOVDD), U9.7 (~{HOLD}), U9.8 (VCC), X1.4 (Vcc); no longer J12.6 (Pin_6), J15.6 (Pin_6)
- net +5V: now also J12.12 (Pin_12), J19.12 (Pin_12), J20.12 (Pin_12)
- net BCLKIN0: now also U6.73 (BCLK_IN0); no longer J12.4 (Pin_4)
- net BCLKIN3: now also J19.7 (Pin_7), U6.84 (BCLK_IN3)
- net GND: now also J12.2 (Pin_2), C1.2, C3.2, C50.2, C52.2, C53.2, C6.2, J19.1 (Pin_1), J19.2 (Pin_2), J20.1 (Pin_1), J20.10 (Pin_10), J20.2 (Pin_2), J20.4 (Pin_4), J20.6 (Pin_6), J20.8 (Pin_8), U6.1 (DGND), U6.18 (PGND), U6.21 (DGND), U6.23 (DGND), U6.29 (DGND), U6.36 (DGND), U6.4 (SPDIFIN), U6.44 (DGND), U6.45 (DGND), U6.5 (SPDIFOUT), U6.66 (DGND), U6.67 (DGND), U6.8 (AGND), U6.88 (DGND), U9.4 (VSS), X1.2 (GND)
- net LRCKIN0: now also U6.74 (LRCLK_IN0/MP10); no longer J12.3 (Pin_3)
- net LRCKIN3: now also J19.5 (Pin_5), U6.85 (LRCLK_IN3/MP13)
- net MCLK: now also J12.3 (Pin_3), J12.4 (Pin_4), J19.3 (Pin_3), J19.4 (Pin_4), J20.3 (Pin_3), U6.27 (CLKOUT); no longer J12.2 (Pin_2)
- net MISO: now also R15.2, U6.38 (MISO/SDA); no longer J15.4 (Pin_4)
- net MOSI: now also R13.2, U6.41 (SS/ADDR0); no longer J15.2 (Pin_2)
- net SCL : now also R17.2, U6.39 (SCLK/SCL); no longer J15.3 (Pin_3)
- net SS: now also R12.2, U6.40 (MOSI/ADDR1); no longer J15.5 (Pin_5)
- net VPP: now also Q1.2 (C), U6.24 (DVDD), U6.43 (DVDD), U6.65 (DVDD), U6.87 (DVDD)
- net ~{RST}: now also U6.28 (RESET)
- net at FER1.1: now also C1.1, C3.1, C48.1, C51.1, U6.19 (PVDD)
- net at FER2.1: now also C50.1, C6.1, U6.9 (AVDD)
- net at JP1.1: now also R11.2, U6.42 (SELFBOOT)
- net ADCIN0 renamed LRCKIN1
- net LRCKIN1: now also U6.77 (LRCLK_IN1/MP11)
- net BCLK0 renamed BCLKOUT0
- net BCLKOUT0: now also U6.48 (BCLK_OUT0)
- net BCLK2 renamed BCLKOUT2
- net BCLKOUT2: now also U6.56 (BCLK_OUT2)
- net LRCLK0 renamed LRCLKOUT0
- net LRCLKOUT0: now also U6.47 (LRCLK_OUT0/MP4)
- net LRCLK2 renamed LRCLKOUT2
- net LRCLKOUT2: now also U6.55 (LRCLK_OUT2/MP8)
- net SDATA0 renamed SDATAOUT0
- net SDATAOUT0: now also U6.49 (SDATA_OUT0)
- net SDATA1+ renamed SDATAOUT1+
- net SDATAOUT1+: now also U6.61 (SDATAIO7/MP23)
- net SDATA2 renamed SDATAOUT2
- net SDATAOUT2: now also U6.57 (SDATA_OUT2)
- net SDATA3+ renamed SDATAOUT3+
- net SDATAOUT3+: now also U6.62 (SDATAIO6/MP22)
- new net: C51.2, R7.2
- new net: U6.25 (XTALIN/MCLK), X1.3 (OUT)
- new net: C48.2, R7.1, U6.20 (PLLFILT)
- new net: Q1.1 (B), R8.1, U6.3 (VDRIVE)
- new net: J7.1 (Pin_1), U6.6 (MP14)
- new net: J7.2 (Pin_2), U6.7 (MP15)
- new net: J21.1 (Pin_1), U6.63 (SDATAIO5/MP21)
- new net: J21.2 (Pin_2), U6.64 (SDATAIO4/MP20)
- new net: J13.1 (Pin_1), U6.69 (SDATAIO3/MP19)
- new net: J13.2 (Pin_2), U6.70 (SDATAIO2/MP18)
- new net: J13.3 (Pin_3), U6.71 (SDATAIO1/MP17)
- new net: J13.4 (Pin_4), U6.72 (SDATAIO0/MP16)
- new net: HL5.1 (K), U6.54 (MP7)
- new net: HL5.2 (A), R14.2
- new net: R10.2, U9.3 (~{WP})
- new net: HL6.2 (A), R16.2
- new net: R9.2, U6.32 (SS_M/MP0), U9.1 (~{CS})
- new net: U6.35 (SDA_M/MISO_M/MP3), U9.2 (SO)
- new net: U6.33 (MOSI_M/MP1), U9.5 (SI)
- new net: U6.34 (SCL_M/SCLK_M/MP2), U9.6 (SCK)
- new net: HL6.1 (K), U6.53 (MP6)
- new net AUXADC0: J15.2 (Pin_2), U6.10 (AUXADC0)
- new net AUXADC1: U6.11 (AUXADC1)
- new net AUXADC2: U6.12 (AUXADC2)
- new net AUXADC3: U6.13 (AUXADC3)
- new net AUXADC4: U6.14 (AUXADC4)
- new net AUXADC5: U6.15 (AUXADC5)
- new net AUXADC6: U6.16 (AUXADC6)
- new net AUXADC7: U6.17 (AUXADC7)
- new net BCLKIN1: J12.7 (Pin_7), U6.76 (BCLK_IN1)
- new net BCLKIN2: J20.7 (Pin_7), U6.81 (BCLK_IN2)
- new net BCLKOUT1: J12.8 (Pin_8), U6.51 (BCLK_OUT1)
- new net BCLKOUT3: J19.8 (Pin_8), U6.59 (BCLK_OUT3)
- new net LRCKIN2: J20.5 (Pin_5), U6.82 (LRCLK_IN2/MP12)
- new net LRCKOUT1: J12.6 (Pin_6), U6.50 (LRCLK_OUT1/MP5)
- new net LRCKOUT3: J19.6 (Pin_6), U6.58 (LRCLK_OUT3/MP9)
- new net SDATAIN0: U6.75 (SDATA_IN0)
- new net SDATAIN1: J12.9 (Pin_9), U6.78 (SDATA_IN1)
- new net SDATAIN2: J20.9 (Pin_9), U6.83 (SDATA_IN2)
- new net SDATAIN3: J19.9 (Pin_9), U6.86 (SDATA_IN3)
- new net SDATAOUT1: J12.10 (Pin_10), U6.52 (SDATA_OUT1)
- new net SDATAOUT3: J19.10 (Pin_10), U6.60 (SDATA_OUT3)
- no-connect marks 23 -> 6
Other:
- note added: "SPM5020T-3R3M-LR"
- moved on the sheet: C10, C100, C11, C12, C13, C14, C15, C17, C18, C19, C20, C21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

Commit message: Промежуточная
Parts:
- added C49: CAP_10n_50V_X7R_0603, Capacitor_SMD:C_0603_1608Metric, symbol Device:C
- added C54, C55, C56, C57: CAP_100n_50V_X7R_0603, Capacitor_SMD:C_0603_1608Metric, symbol Device:C
- FER1, FER2: footprint Resistor_SMD:R_0805_2012Metric_Pad1.15x1.40mm_HandSolder -> Resistor_SMD:R_0805_2012Metric_Pad1.20x1.40mm_HandSolder
- J15: footprint Connector_JST:JST_XH_B6B-XH-A_1x06_P2.50mm_Vertical -> Connector_JST:JST_XH_B3B-XH-A_1x03_P2.50mm_Vertical
- J18, J6: value Out -> DEGSON 2604 8x5; footprint my:DG16S-B-08P-13-00A(H) -> Connector_Degson:DEGSON_8x5
- JP1: footprint Resistor_SMD:R_0603_1608Metric_Pad1.05x0.95mm_HandSolder -> Resistor_SMD:R_0603_1608Metric_Pad0.98x0.95mm_HandSolder
Connections:
- net GND: now also C49.2, C54.2, C55.2, C56.2, C57.2; no longer J20.4 (Pin_4), J20.8 (Pin_8), U6.4 (SPDIFIN), U6.5 (SPDIFOUT)
- net SCL: no longer R5.2, U4.21 (SDA), U8.21 (SDA)
- net VPP: now also C49.1, C54.1, C55.1, C56.1, C57.1
- net AUXADC1: no longer names the net of U6.11 (AUXADC1)
- net AUXADC2: no longer names the net of U6.12 (AUXADC2)
- net AUXADC3: no longer names the net of U6.13 (AUXADC3)
- net AUXADC4: no longer names the net of U6.14 (AUXADC4)
- net AUXADC5: no longer names the net of U6.15 (AUXADC5)
- net AUXADC6: no longer names the net of U6.16 (AUXADC6)
- net AUXADC7: no longer names the net of U6.17 (AUXADC7)
- net ~{RST} renamed RST
- new net SDA: R5.2, U4.21 (SDA), U8.21 (SDA)
- new net SPDIFIN: J20.4 (Pin_4), U6.4 (SPDIFIN)
- new net SPDIFOUT: J20.8 (Pin_8), U6.5 (SPDIFOUT)
- no-connect marks 6 -> 13

Commit message: Почти все
Parts:
- J13: footprint Connector_PinHeader_2.54mm:PinHeader_1x04_P2.54mm_Vertical -> Connector_PinHeader_2.54mm:PinHeader_1x05_P2.54mm_Vertical; symbol AMPP_1466_V0-rescue:Conn_01x04_Male-Connector -> Connector:Conn_01x05_Pin
- J21, J7: footprint Connector_PinHeader_2.54mm:PinHeader_1x02_P2.54mm_Vertical -> Connector_PinHeader_2.54mm:PinHeader_1x03_P2.54mm_Vertical; symbol AMPP_1466_V0-rescue:Conn_01x02_Male-Connector -> Connector:Conn_01x03_Pin
Connections:
- net GND: now also J13.5 (Pin_5), J21.3 (Pin_3), J7.3 (Pin_3), U6.89 (GND)
- net at J13.1 (Pin_1): now also U6.72 (SDATAIO0/MP16); no longer U6.69 (SDATAIO3/MP19)
- net at J13.2 (Pin_2): now also U6.71 (SDATAIO1/MP17); no longer U6.70 (SDATAIO2/MP18)
- net at J13.3 (Pin_3): now also U6.70 (SDATAIO2/MP18); no longer U6.71 (SDATAIO1/MP17)
- net at J13.4 (Pin_4): now also U6.69 (SDATAIO3/MP19); no longer U6.72 (SDATAIO0/MP16)
Changed lines of the file:
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@@
     (stroke (width 0) (type default))
   )
+  (wire (pts (xy 106.045 62.865) (xy 108.585 62.865))
+    (stroke (width 0) (type default))
+  )
   (wire (pts (xy 130.81 146.685) (xy 148.59 146.685))
     (stroke (width 0) (type default))
@@
     (stroke (width 0) (type default))
   )
-  (wire (pts (xy 93.98 90.805) (xy 102.87 90.805))
+  (wire (pts (xy 81.28 90.805) (xy 102.87 90.805))
     (stroke (width 0) (type default))
   )
@@
     (stroke (width 0) (type default))
   )
+  (wire (pts (xy 200.025 76.835) (xy 200.025 78.105))
+    (stroke (width 0) (type default))
+  )
   (wire (pts (xy 55.245 210.185) (xy 58.42 210.185))
     (stroke (width 0) (type default))
@@
     (stroke (width 0) (type default))
   )
-  (wire (pts (xy 93.98 88.265) (xy 102.87 88.265))
+  (wire (pts (xy 81.28 88.265) (xy 102.87 88.265))
     (stroke (width 0) (type default))
   )
@@
     (stroke (width 0) (type default))
   )
+  (wire (pts (xy 166.37 47.625) (xy 168.275 47.625))
+    (stroke (width 0) (type default))
+  )
   (wire (pts (xy 234.95 151.765) (xy 234.95 153.035))
     (stroke (width 0) (type default))
@@
     (stroke (width 0) (type default))
   )
+  (wire (pts (xy 81.28 93.345) (xy 83.185 93.345))
+    (stroke (width 0) (type default))
+  )
   (wire (pts (xy 345.44 114.3) (xy 349.25 114.3))
     (stroke (width 0) (type default))
@@
     )
   )
-  (symbol (lib_id "AMPP_1466_V0-rescue:Conn_01x02_Male-Connector") (at 88.9 88.265 0) (unit 1)
+  (symbol (lib_id "Connector:Conn_01x03_Pin") (at 76.2 90.805 0) (unit 1)
     (in_bom yes) (on_board yes) (dnp no)
-    (property "Reference" "J7" (at 90.805 92.71 0)
+    (property "Reference" "J7" (at 78.105 95.25 0)
       (effects (font (size 0.63 0.63)))
     )
-    (property "Value" "Conn_01x02_Male" (at 91.6432 85.979 0)
+    (property "Value" "Conn_01x02_Male" (at 78.9432 88.519 0)
       (effects (font (size 0.63 0.63)) hide)
     )
-    (property "Footprint" "Connector_PinHeader_2.54mm:PinHeader_1x02_P2.54mm_Vertical" (at 88.9 88.265 0)
+    (property "Footprint" "Connector_PinHeader_2.54mm:PinHeader_1x03_P2.54mm_Vertical" (at 76.2 90.805 0)
       (effects (font (size 1.27 1.27)) hide)
     )
-    (property "Datasheet" "~" (at 88.9 88.265 0)
+    (property "Datasheet" "~" (at 76.2 90.805 0)
       (effects (font (size 1.27 1.27)) hide)
     )
     (pin "1")
     (pin "2")
+    (pin "3")
     (instances
       (project "Amplifier"
@@
     )
   )
-  (symbol (lib_id "AMPP_1466_V0-rescue:Conn_01x02_Male-Connector") (at 205.105 83.185 180) (unit 1)
+  (symbol (lib_id "Connector:Conn_01x03_Pin") (at 205.105 80.645 180) (unit 1)
     (in_bom yes) (on_board yes) (dnp no)
-    (property "Reference" "J21" (at 207.645 81.915 0)
+    (property "Reference" "J21" (at 207.645 79.375 0)
       (effects (font (size 0.63 0.63)))
     )
-    (property "Value" "Conn_01x02_Male" (at 202.3618 85.471 0)
+    (property "Value" "Conn_01x02_Male" (at 202.3618 82.931 0)
       (effects (font (size 0.63 0.63)) hide)
     )
-    (property "Footprint" "Connector_PinHeader_2.54mm:PinHeader_1x02_P2.54mm_Vertical" (at 205.105 83.185 0)
+    (property "Footprint" "Connector_PinHeader_2.54mm:PinHeader_1x03_P2.54mm_Vertical" (at 205.105 80.645 0)
       (effects (font (size 1.27 1.27)) hide)
     )
-    (property "Datasheet" "~" (at 205.105 83.185 0)
+    (property "Datasheet" "~" (at 205.105 80.645 0)
       (effects (font (size 1.27 1.27)) hide)
     )
     (pin "1")
     (pin "2")
+    (pin "3")
     (instances
       (project "daw00"
@@
     )
   )
-  (symbol (lib_id "AMPP_1466_V0-rescue:Conn_01x04_Male-Connector") (at 161.29 42.545 270) (unit 1)
+  (symbol (lib_id "Connector:Conn_01x05_Pin") (at 161.29 42.545 90) (mirror x) (unit 1)
     (in_bom yes) (on_board yes) (dnp no)
-    (property "Reference" "J13" (at 160.02 40.64 90)
+    (property "Reference" "J13" (at 162.56 40.64 90)
       (effects (font (size 0.63 0.63)) (justify left))
     )
-    (property "Value" "Conn_01x04_Male" (at 160.6042 41.8338 0)
+    (property "Value" "Conn_01x04_Male" (at 161.9758 41.8338 0)
       (effects (font (size 0.63 0.63)) (justify right) hide)
     )
-    (property "Footprint" "Connector_PinHeader_2.54mm:PinHeader_1x04_P2.54mm_Vertical" (at 161.29 42.545 0)
+    (property "Footprint" "Connector_PinHeader_2.54mm:PinHeader_1x05_P2.54mm_Vertical" (at 161.29 42.545 0)
       (effects (font (size 1.27 1.27)) hide)
     )
@@
     (pin "3")
     (pin "4")
+    (pin "5")
     (instances
       (project "Amplifier"
@@
     )
   )
+  (symbol (lib_id "AMPP_1466_V0-rescue:GND-power") (at 168.275 47.625 90) (unit 1)
+    (in_bom yes) (on_board yes) (dnp no)
+    (property "Reference" "#PWR035" (at 174.625 47.625 0)
+      (effects (font (size 0.63 0.63)) hide)
+    )
+    (property "Value" "GND" (at 172.6692 47.498 0)
+      (effects (font (size 0.63 0.63)))
+    )
+    (property "Footprint" "" (at 168.275 47.625 0)
+      (effects (font (size 1.27 1.27)) hide)
+    )
+    (property "Datasheet" "" (at 168.275 47.625 0)
+      (effects (font (size 1.27 1.27)) hide)
+    )
+    (pin "1")
+    (instances
+      (project "daw00"
+        (path "/ca4cfd42-59e1-4265-8267-972d6aaac6ff/4aeb4b63-8869-4af7-96e8-06e4a551ac30"
+          (reference "#PWR035") (unit 1)
+        )
+      )
+    )
+  )
   (symbol (lib_id "RDC4-0027v1-rescue:CON_JUMPER-rk-infinitas-rescue-SigmaDSP-ADAU1452-rescue-SigmaDSP-ADAU1452-rescue-SigmaDSP-ADAU1452-rescue") (at 201.295 146.05 270) (unit 1)
     (in_bom yes) (on_board yes) (dnp no)
@@
     )
   )
+  (symbol (lib_id "AMPP_1466_V0-rescue:GND-power") (at 200.025 76.835 180) (unit 1)
+    (in_bom yes) (on_board yes) (dnp no)
+    (property "Reference" "#PWR034" (at 200.025 70.485 0)
+      (effects (font (size 0.63 0.63)) hide)
+    )
+    (property "Value" "GND" (at 199.898 72.4408 0)
+      (effects (font (size 0.63 0.63)))
+    )
+    (property "Footprint" "" (at 200.025 76.835 0)
+      (effects (font (size 1.27 1.27)) hide)
+    )
+    (property "Datasheet" "" (at 200.025 76.835 0)
+      (effects (font (size 1.27 1.27)) hide)
+    )
+    (pin "1")
+    (instances
+      (project "daw00"
+        (path "/ca4cfd42-59e1-4265-8267-972d6aaac6ff/4aeb4b63-8869-4af7-96e8-06e4a551ac30"
+          (reference "#PWR034") (unit 1)
+        )
+      )
+    )
+  )
+  (symbol (lib_id "AMPP_1466_V0-rescue:GND-power") (at 106.045 62.865 270) (unit 1)
+    (in_bom yes) (on_board yes) (dnp no)
+    (property "Reference" "#PWR052" (at 99.695 62.865 0)
+      (effects (font (size 0.63 0.63)) hide)
+    )
+    (property "Value" "GND" (at 101.6508 62.992 0)
+      (effects (font (size 0.63 0.63)))
+    )
+    (property "Footprint" "" (at 106.045 62.865 0)
+      (effects (font (size 1.27 1.27)) hide)
+    )
+    (property "Datasheet" "" (at 106.045 62.865 0)
+      (effects (font (size 1.27 1.27)) hide)
+    )
+    (pin "1")
+    (instances
+      (project "daw00"
+        (path "/ca4cfd42-59e1-4265-8267-972d6aaac6ff/4aeb4b63-8869-4af7-96e8-06e4a551ac30"
+          (reference "#PWR052") (unit 1)
+        )
+      )
+    )
+  )
   (symbol (lib_id "power:GND") (at 101.6 264.16 0) (unit 1)
     (in_bom yes) (on_board yes) (dnp no)
@@
     )
   )
+  (symbol (lib_id "power:GND") (at 83.185 93.345 90) (unit 1)
+    (in_bom yes) (on_board yes) (dnp no)
+    (property "Reference" "#PWR050" (at 89.535 93.345 0)
+      (effects (font (size 0.63 0.63)) hide)
+    )
+    (property "Value" "GND" (at 86.995 93.345 0)
+      (effects (font (size 0.63 0.63)))
+    )
+    (property "Footprint" "" (at 83.185 93.345 0)
+      (effects (font (size 1.27 1.27)))
+    )
+    (property "Datasheet" "" (at 83.185 93.345 0)
+      (effects (font (size 1.27 1.27)))
+    )
+    (pin "1")
+    (instances
+      (project "daw00"
+        (path "/ca4cfd42-59e1-4265-8267-972d6aaac6ff/4aeb4b63-8869-4af7-96e8-06e4a551ac30"
+          (reference "#PWR050") (unit 1)
+        )
+      )
+    )
+  )
   (symbol (lib_id "AMPP_1466_V0-rescue:+5V-power") (at 74.93 222.885 180) (unit 1)
     (in_bom yes) (on_board yes) (dnp no)
@@
     (pin "88")
     (pin "9")
+    (pin "89")
     (instances
       (project "Amplifier"

Commit message: Основная плата все
Parts:
- C1, C6: value CAP_10u0_25V_X5R_0805 -> CAP_10u0_50V_X7R_1206; footprint Capacitor_SMD:C_0805_2012Metric -> Capacitor_SMD:C_1206_3216Metric
- J12, J19, J20: value Conn_01x06_Male -> Conn_edge_2x6_2.54_Male

Commit message: Почти все
Parts:
- C1, C6: Value1 10u0 -> 10u
- C10, C11, C12, C13, C14, C23, C24, C25, C26, C27, C28, C29, C30, C65, C66, C67, C68, C69, C77, C78, C79, C80, C81, C82, C83, C84: value 1,0uF -> CAP_1u_50V_X7R_0603; Value1 (none) -> 1u
- C100, C39, C40, C41, C42, C43, C44, C45, C46, C93, C94, C95, C96, C97, C98, C99: value 10n -> CAP_10n_50V_X7R_0603; Value1 (none) -> 10n
- C15, C18, C19, C22, C70, C72, C73, C76: value 100n -> CAP_100n_50V_X7R_0603; Value1 (none) -> 100n
- C17, C20, C21, C47, C64, C71, C74, C75: value 10,0uF -> CAP_10u0_50V_X7R_1206; Value1 (none) -> 10u
- C31, C32, C33, C34, C35, C36, C37, C38, C85, C86, C87, C88, C89, C90, C91, C92: value 1.0uF -> CAP_1u_50V_X7R_0603; footprint Capacitor_SMD:C_0805_2012Metric -> Capacitor_SMD:C_0603_1608Metric; Value1 (none) -> 1u
- C52: value CAP_10n_25V_X7R_0603 -> CAP_10n_50V_X7R_0603
- L1, L10, L11, L12, L13, L14, L15, L16, L2, L3, L4, L5, L6, L7, L8, L9: value 3.3uH -> 3u3; MP ETQP3M3R3KVP -> (none); Value1 (none) -> SPM4020T-3R3M-LR
- R10, R11, R12, R13, R15, R17, R9: value RES_10K0_1%_0.125W_Thick_0603 -> 10k
- R14, R16: value RES_51R0_1%_0.125W_Thick_0603 -> 510
- R22, R4, R5: value 4k7 -> 4.7K
- R7: value RES_4K3_1%_0.125W_Thick_0603 -> 4.3K
- R8: value RES_1K0_1%_0.125W_Thick_0603 -> 1k
