File: daw00/computer.kicad_sch (KiCad schematic)
At the start: 18 parts, among them J2 USB_A_Stacked, J3 UART, J4 SWD, U10 STM32F030F4Px, U12 Nanopi NEO Air, U14 PC357, U3 TPS3828-33DBVT

Commit message: Промежуточная
Parts:
- removed C16: 2n2, Capacitor_SMD:C_0603_1608Metric, symbol AMPP_1466_V0-rescue:C_micro-my
- removed R24: 47K, Resistor_SMD:R_0603_1608Metric, symbol AMPP_1466_V0-rescue:R_micro-my
- removed R42: 10K, Resistor_SMD:R_0603_1608Metric, symbol AMPP_1466_V0-rescue:R_Small-my
- removed R43: 1.2k, Resistor_SMD:R_0805_2012Metric, symbol Источник-24в-на-SG3525-rescue:R_Small-my
- removed U14: PC357, spacestudio:4pin_mini_flat, symbol Isolator:PC817
- removed VD1: diode BAS85.115, w_smd_diode:sod80c, symbol AMPP_1466_V0-rescue:D_Small-my
- J2: footprint Connector_USB:USB_A_CUI_UJ2-ADH-TH_Horizontal_Stacked -> 00-mylib:USB_A_STACKED
- J4: footprint Connector_JST:JST_XH_B4B-XH-A_1x04_P2.50mm_Vertical -> Connector_PinHeader_2.54mm:PinHeader_1x03_P2.54mm_Vertical; symbol AMPP_1466_V0-rescue:Conn_01x04-Connector_Generic -> Connector_Generic:Conn_01x03
Connections:
- net ~{RST} is gone; now on an unnamed net: R1.2, U3.1 (~{RESET})
- net RST: no longer names the net of U10.4 (NRST)
- net RST: no longer J4.4 (Pin_4)
- no-connect marks 4 -> 30

Commit message: Почти все
Connections:
- net RST: now reaches R1.2, U10.4 (NRST), U3.1 (~{RESET})
Changed lines of the file:
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@@
   (junction (at 60.96 64.77) (diameter 0) (color 0 0 0 0)
+  )
+  (junction (at 189.23 53.975) (diameter 0) (color 0 0 0 0)
   )
   (junction (at 193.04 74.295) (diameter 0) (color 0 0 0 0)
@@
     (stroke (width 0) (type default))
   )
+  (wire (pts (xy 189.23 53.975) (xy 203.2 53.975))
+    (stroke (width 0) (type default))
+  )
   (wire (pts (xy 60.96 77.47) (xy 77.47 77.47))
     (stroke (width 0) (type default))
@@
     (stroke (width 0) (type default))
   )
-  (wire (pts (xy 179.07 53.975) (xy 203.2 53.975))
+  (wire (pts (xy 179.07 53.975) (xy 189.23 53.975))
+    (stroke (width 0) (type default))
+  )
+  (wire (pts (xy 189.23 50.8) (xy 189.23 53.975))
     (stroke (width 0) (type default))
   )
@@
     )
   )
+  (global_label "RST" (shape input) (at 189.23 50.8 90) (fields_autoplaced)
+    (effects (font (size 1.27 1.27)) (justify left))
+    (property "Intersheetrefs" "${INTERSHEET_REFS}" (at 189.23 44.3677 90)
+      (effects (font (size 1.27 1.27)) (justify left) hide)
+    )
+  )

Commit message: Основная плата все
Connections:
- net REMOTE: now also U12.7 (GPIO_G11); no longer U10.10 (PA4)
- net ACC_IN: now reaches U12.12 (GPIO_A6)
- no-connect marks 30 -> 29
Other:
- moved on the sheet: C5, C9, J4, R1, R23, R6, TP1, U10, U3

Commit message: Почти все
Parts:
- C9: value 100n -> CAP_100n_50V_X7R_0603; Value1 (none) -> 100n
