File: daw00/power.kicad_sch (KiCad schematic)
At the start: 74 parts, among them J1 Power in, J10 +6V, J11 GND, J14 +24V, J16 GND, J22 Power, J5 +6V, U1 L78L18_SOT89, U13 SG3525, U15 MOC3023M, U16 MOC3023M, U2 LD1086D2T33TR, U7 LP2985-5.0

Commit message: Промежуточная
Parts:
- removed J1: Power in, my:DG16S-B-02P-13-00A(H), symbol AMPP_1466_V0-rescue:Screw_Terminal_01x02-Connector
- removed J5: +6V, TerminalBlock_Phoenix:TerminalBlock_Phoenix_MKDS-1,5-2-5.08_1x02_P5.08mm_Horizontal, symbol AMPP_1466_V0-rescue:Screw_Terminal_01x02-Connector
- added F1: Fuse, 00-mylib:Fuse_Blade_vertical, symbol Device:Fuse
- added J8: DEGSON 2604 1x5, Connector_Degson:DEGSON_1x5, symbol Connector_Generic:Conn_01x01
- added VD1: SS56, Diode_SMD:D_SMC, symbol Источник-24в-на-SG3525-rescue:D_Small-my
- J10, J11: footprint Connector_Wire:SolderWirePad_1x01_Drill2mm -> TestPoint:TestPoint_Pad_1.5x1.5mm
- J14, J16: footprint Connector_Wire:SolderWirePad_1x01_Drill2.5mm -> TestPoint:TestPoint_Pad_1.5x1.5mm
- J22: value Power -> KF206-7.5-2P; footprint (none) -> Connector_Degson:DEGSON_2x7.5; symbol Connector_Generic:Conn_01x03 -> Connector_Generic:Conn_01x02
- L19: footprint my:L_Axial_L24.0mm_D7.5mm_P27.94mm_Horizontal_Fastron_MESC -> my:L_Axial_L26.0mm_D9.0mm_P5.08mm_Vertical
Connections:
- net +6V: now also C113.1, J10.1 (Pin_1), VD10.1 (K), VD12.1 (K)
- net +BATT: now also F1.1; no longer L18.1
- net ACC: now also J8.1 (Pin_1); no longer J22.2 (Pin_2)
- net GND: now also U16.2; no longer U16.1
- net GNDPWR: now also J22.2 (Pin_2), VD1.2 (A); no longer J22.3 (Pin_3)
- net at R45.2: now also U16.1; no longer U16.2
- new net: F1.2, L18.1, VD1.1 (K)
Other:
- moved on the sheet: R45

Commit message: Почти все
Parts:
- TR1: footprint my:Trans10_Toroid_Horizontal_D60mm -> 00-mylib:Transformer_ETD44_Horizontal
- U15, U16: value MOC3023M -> PC817; footprint Package_DIP:DIP-6_W7.62mm -> Package_DIP:DIP-4_W7.62mm; symbol Relay_SolidState:MOC3023M -> PCM_Optocoupler_AKL:PC817
Connections:
- net at U16.3: now also VD15.1 (K)
- net at U16.4: now also C105.1, R29.1, U15.3; no longer VD15.1 (K)
- net at VD14.1 (K): now also U15.4; no longer U15.6
Changed lines of the file:
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@@
+    (stroke (width 0) (type default))
+  )
+  (wire (pts (xy 99.06 45.085) (xy 102.87 45.085))
+    (stroke (width 0) (type default))
+  )
+  (wire (pts (xy 99.06 55.245) (xy 102.87 55.245))
     (stroke (width 0) (type default))
   )
@@
     (stroke (width 0) (type default))
   )
+  (wire (pts (xy 114.3 55.245) (xy 114.3 52.705))
+    (stroke (width 0) (type default))
+  )
   (wire (pts (xy 167.64 118.11) (xy 170.18 118.11))
     (stroke (width 0) (type default))
@@
     (stroke (width 0) (type default))
   )
+  (wire (pts (xy 110.49 45.085) (xy 114.3 45.085))
+    (stroke (width 0) (type default))
+  )
   (wire (pts (xy 41.91 173.355) (xy 41.91 172.085))
     (stroke (width 0) (type default))
@@
     (stroke (width 0) (type default))
   )
+  (wire (pts (xy 67.31 55.245) (xy 71.12 55.245))
+    (stroke (width 0) (type default))
+  )
   (wire (pts (xy 147.32 172.085) (xy 140.97 172.085))
     (stroke (width 0) (type default))
   )
+  (wire (pts (xy 71.12 55.245) (xy 71.12 52.705))
+    (stroke (width 0) (type default))
+  )
   (wire (pts (xy 137.16 64.135) (xy 140.97 64.135))
     (stroke (width 0) (type default))
@@
     (stroke (width 0) (type default))
   )
+  (wire (pts (xy 55.88 52.705) (xy 55.88 55.245))
+    (stroke (width 0) (type default))
+  )
   (wire (pts (xy 115.57 118.11) (xy 118.11 118.11))
     (stroke (width 0) (type default))
@@
     (stroke (width 0) (type default))
   )
+  (wire (pts (xy 71.12 45.085) (xy 71.12 47.625))
+    (stroke (width 0) (type default))
+  )
   (wire (pts (xy 33.02 182.245) (xy 41.91 182.245))
     (stroke (width 0) (type default))
@@
     (stroke (width 0) (type default))
   )
+  (wire (pts (xy 55.88 55.245) (xy 59.69 55.245))
+    (stroke (width 0) (type default))
+  )
   (wire (pts (xy 44.45 106.68) (xy 44.45 116.84))
     (stroke (width 0) (type default))
@@
     (stroke (width 0) (type default))
   )
+  (wire (pts (xy 114.3 45.085) (xy 114.3 47.625))
+    (stroke (width 0) (type default))
+  )
   (wire (pts (xy 165.1 118.11) (xy 167.64 118.11))
     (stroke (width 0) (type default))
@@
     (stroke (width 0) (type default))
   )
+  (wire (pts (xy 110.49 55.245) (xy 114.3 55.245))
+    (stroke (width 0) (type default))
+  )
   (wire (pts (xy 45.72 88.9) (xy 48.26 88.9))
     (stroke (width 0) (type default))
@@
     (stroke (width 0) (type default))
   )
+  (wire (pts (xy 67.31 45.085) (xy 71.12 45.085))
+    (stroke (width 0) (type default))
+  )
   (wire (pts (xy 123.19 88.265) (xy 124.46 88.265))
     (stroke (width 0) (type default))
@@
     (stroke (width 0) (type default))
   )
+  (wire (pts (xy 55.88 47.625) (xy 55.88 45.085))
+    (stroke (width 0) (type default))
+  )
   (wire (pts (xy 163.83 114.935) (xy 166.37 114.935))
     (stroke (width 0) (type default))
   )
+  (wire (pts (xy 99.06 47.625) (xy 99.06 45.085))
+    (stroke (width 0) (type default))
+  )
   (wire (pts (xy 41.91 104.14) (xy 41.91 101.6))
     (stroke (width 0) (type default))
@@
     (stroke (width 0) (type default))
   )
+  (wire (pts (xy 55.88 45.085) (xy 59.69 45.085))
+    (stroke (width 0) (type default))
+  )
   (wire (pts (xy 187.96 93.98) (xy 194.31 93.98))
     (stroke (width 0) (type default))
@@
   )
   (wire (pts (xy 180.34 169.545) (xy 190.5 169.545))
+    (stroke (width 0) (type default))
+  )
+  (wire (pts (xy 99.06 52.705) (xy 99.06 55.245))
     (stroke (width 0) (type default))
   )
@@
     )
   )
-  (symbol (lib_id "Relay_SolidState:MOC3023M") (at 106.68 50.165 180) (unit 1)
-    (in_bom yes) (on_board yes) (dnp no) (fields_autoplaced)
-    (property "Reference" "U16" (at 106.68 41.275 0)
-      (effects (font (size 0.63 0.63)))
-    )
-    (property "Value" "MOC3023M" (at 106.68 43.815 0)
-      (effects (font (size 0.63 0.63)))
-    )
-    (property "Footprint" "Package_DIP:DIP-6_W7.62mm" (at 111.76 45.085 0)
+  (symbol (lib_id "PCM_Optocoupler_AKL:PC817") (at 106.68 50.165 180) (unit 1)
+    (in_bom yes) (on_board yes) (dnp no)
+    (property "Reference" "U16" (at 105.41 43.815 0)
+      (effects (font (size 0.63 0.63)) (justify right))
+    )
+    (property "Value" "PC817" (at 105.41 45.085 0)
+      (effects (font (size 0.63 0.63)) (justify right))
+    )
+    (property "Footprint" "Package_DIP:DIP-4_W7.62mm" (at 100.33 51.435 0)
       (effects (font (size 1.27 1.27) italic) (justify left) hide)
     )
-    (property "Datasheet" "https://www.onsemi.com/pub/Collateral/MOC3023M-D.PDF" (at 106.68 50.165 0)
+    (property "Datasheet" "https://www.tme.eu/Document/7534c9f89aa4b1eba4ec90182e378328/PC817_2_3_47.pdf" (at 106.68 50.165 0)
       (effects (font (size 1.27 1.27)) (justify left) hide)
     )
-    (pin "5")
     (pin "3")
-    (pin "6")
     (pin "4")
     (pin "1")
@@
     )
   )
-  (symbol (lib_id "Relay_SolidState:MOC3023M") (at 63.5 50.165 0) (unit 1)
-    (in_bom yes) (on_board yes) (dnp no) (fields_autoplaced)
-    (property "Reference" "U15" (at 63.5 41.783 0)
-      (effects (font (size 0.63 0.63)))
-    )
-    (property "Value" "MOC3023M" (at 63.5 44.323 0)
-      (effects (font (size 0.63 0.63)))
-    )
-    (property "Footprint" "Package_DIP:DIP-6_W7.62mm" (at 58.42 55.245 0)
+  (symbol (lib_id "PCM_Optocoupler_AKL:PC817") (at 63.5 50.165 0) (unit 1)
+    (in_bom yes) (on_board yes) (dnp no)
+    (property "Reference" "U15" (at 61.595 44.45 0)
+      (effects (font (size 0.63 0.63)) (justify left))
+    )
+    (property "Value" "PC817" (at 61.595 45.72 0)
+      (effects (font (size 0.63 0.63)) (justify left))
+    )
+    (property "Footprint" "Package_DIP:DIP-4_W7.62mm" (at 69.85 48.895 0)
       (effects (font (size 1.27 1.27) italic) (justify left) hide)
     )
-    (property "Datasheet" "https://www.onsemi.com/pub/Collateral/MOC3023M-D.PDF" (at 63.5 50.165 0)
+    (property "Datasheet" "https://www.tme.eu/Document/7534c9f89aa4b1eba4ec90182e378328/PC817_2_3_47.pdf" (at 63.5 50.165 0)
       (effects (font (size 1.27 1.27)) (justify left) hide)
     )
-    (pin "5")
     (pin "3")
-    (pin "6")
     (pin "4")
     (pin "1")
@@
       (effects (font (size 0.63 0.63)))
     )
-    (property "Footprint" "my:Trans10_Toroid_Horizontal_D60mm" (at 148.59 95.25 0)
+    (property "Footprint" "00-mylib:Transformer_ETD44_Horizontal" (at 148.59 95.25 0)
       (effects (font (size 1.27 1.27)) hide)
     )
@@
   (symbol (lib_id "Источник-24в-на-SG3525-rescue:R_Small-my") (at 118.745 52.705 270) (unit 1)
     (in_bom yes) (on_board yes) (dnp no)
-    (property "Reference" "R45" (at 115.951 50.419 90)
-      (effects (font (size 0.63 0.63)))
-    )
-    (property "Value" "330" (at 120.777 50.419 90)
+    (property "Reference" "R45" (at 118.745 51.435 90)
+      (effects (font (size 0.63 0.63)))
+    )
+    (property "Value" "330" (at 121.285 51.435 90)
       (effects (font (size 0.63 0.63)))
     )
@@
       (effects (font (size 0.63 0.63)))
     )
-    (property "Value" "1N5819" (at 98.044 45.085 0)
-      (effects (font (size 0.63 0.63)))
-    )
+    (property "Value" "1N5819" (at 95.25 45.085 0)
+      (effects (font (size 0.63 0.63)))
+    )

Commit message: Основная плата все
Parts:
- added C16: CAP_10u0_50V_X7R_1206, Capacitor_SMD:C_1206_3216Metric, symbol Источник-24в-на-SG3525-rescue:C_Small-my
- added R18, R43: 4.7k, Resistor_SMD:R_0603_1608Metric, symbol Источник-24в-на-SG3525-rescue:R_Small-my
- added R19: 10k, Resistor_SMD:R_0603_1608Metric, symbol Источник-24в-на-SG3525-rescue:R_Small-my
- added R24: 1k, Resistor_SMD:R_0603_1608Metric, symbol Источник-24в-на-SG3525-rescue:R_Small-my
- added R42: 1.2k, Resistor_SMD:R_1206_3216Metric, symbol Источник-24в-на-SG3525-rescue:R_Small-my
- added U5: TLP627, Package_DIP:DIP-4_W7.62mm, symbol Isolator:TLP627
- C102, C111: value 1n -> CAP_1n_50V_X7R_0603; footprint Capacitor_SMD:C_0805_2012Metric -> Capacitor_SMD:C_0603_1608Metric; Value1 (none) -> 1n
- C103, C106: value 10n -> CAP_10n_50V_X7R_0603; footprint Capacitor_SMD:C_0805_2012Metric -> Capacitor_SMD:C_0603_1608Metric; Value1 (none) -> 10n
- C104: value 2.2μ -> CAP_2u2_50V_X7R_1206; Value1 (none) -> 2.2u
- C105, C125: value 10μ -> CAP_10u0_50V_X7R_1206; Value1 (none) -> 10u
- C109, C110: value 22n -> CAP_22n_50V_X7R_0603; footprint Capacitor_SMD:C_0805_2012Metric -> Capacitor_SMD:C_0603_1608Metric; Value1 (none) -> 22n
- C112: value 100n -> CAP_100n_50V_X7R_0603; footprint Capacitor_SMD:C_0805_2012Metric -> Capacitor_SMD:C_0603_1608Metric; Value1 (none) -> 100n
- C63: footprint Capacitor_SMD:C_0805_2012Metric -> Capacitor_SMD:C_1206_3216Metric
- R25, R26, R27, R28, R29, R30, R31, R32, R33, R34, R35, R39: footprint Resistor_SMD:R_0805_2012Metric -> Resistor_SMD:R_0603_1608Metric
- R41: footprint Resistor_SMD:R_0805_2012Metric -> Resistor_SMD:R_1206_3216Metric
- R45: value 330 -> 1k; footprint Resistor_SMD:R_0805_2012Metric -> Resistor_SMD:R_0603_1608Metric
- U15, U16: value PC817 -> TLP627; symbol PCM_Optocoupler_AKL:PC817 -> Isolator:TLP627
- VD2: footprint w_smd_diode:do214ac -> Diode_SMD:D_SMA
Connections:
- net +3V3: now also U5.4
- net ACC: now also R42.2
- net GND: now also R19.2
- net GNDPWR: now also C16.2, R18.2, R43.2, U5.2
- net at C107.1, C108.1, C109.2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: now also U15.4, U16.4; no longer VD14.2 (A), VD15.2 (A)
- net at U16.3: now also VD15.2 (A), R43.1; no longer VD15.1 (K)
- net at C105.1, R29.1: now also VD14.1 (K), VD15.1 (K); no longer U15.3, U16.4
- new net: R18.1, U15.3, VD14.2 (A)
- new net: C16.1, R42.1, U5.1
- new net: R19.1, R24.1, U5.3
- new net ACC_IN: R24.2
Other:
- moved on the sheet: C104, C106, C107, C108, C110, C113, C125, C2, C4, C60, C61, C62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

Commit message: Почти все
Parts:
- C107, C108: Value1 (none) -> 2200u
- C113, C114, C115: value 330μ -> CAP_330μ_35V; Value1 (none) -> 330u
- C2, C7: value 0,33uF -> CAP_330n_50V_X7R_0603; Value1 (none) -> 330n
- C4, C60, C62, C8: value 100n -> CAP_100n_50V_X7R_0603; Value1 (none) -> 100n
- C61: value 10n -> CAP_10n_50V_X7R_0603; Value1 (none) -> 10n
- C63: value 10,0uF -> CAP_10u0_50V_X7R_1206; Value1 (none) -> 10u
- L19: footprint my:L_Axial_L26.0mm_D9.0mm_P5.08mm_Vertical -> 00-mylib:L_Toroid_Vertical_L33.0mm_W17.8mm_P12.70mm_Pulse_KM-5
- R18, R43: value 4.7k -> 4.7K
