File: daw00/daw00.kicad_pcb (KiCad board)
At the start: 2 copper layers, 149.9 x 171.2 mm, 232 parts, among them J10 +6V, J11 GND, J12 Conn_01x06_Male, J13 Conn_01x04_Male, J14 +24V, J15 Volume, J16 GND, J18 DEGSON 2604 8x5, J19 Conn_01x06_Male, J2 USB_A_Stacked, J20 Conn_01x06_Male, J21 Conn_01x02_Male, J22 KF206-7.5-2P, J3 UART, J4 SWD, J6 DEGSON 2604 8x5, J7 Conn_01x02_Male, J8 DEGSON 2604 1x5, Q1 2STF2360, U1 L78L18_SOT89, U10 STM32F030F4Px, U12 Nanopi NEO Air, U13 SG3525, U15 MOC3023M, U16 MOC3023M, U2 LD1086D2T33TR, U3 TPS3828-33DBVT, U4 TAS6424QDKQRQ1, U6 ADAU1467WBCPZ300RL, U7 LP2985-5.0, U8 TAS6424QDKQRQ1, U9 25AA1024-I/SM, X1 SG-8002CA 24.5760M-PCBL3

Commit message: next
Parts:
- moved C50 2.67 mm to (34.0, 89.3)
- moved C6 2.67 mm to (35.8, 89.5)
- moved FER2 2.67 mm to (37.8, 89.8)
- moved J4 1.52 mm to (71.2, 106.6)
Routing:
- net SCL: track 2.67 -> 131.7 mm, vias 0 -> 3
- net SDA: track 2.89 -> 123.3 mm, vias 0 -> 3
- net Mute: track 6.00 -> 125.8 mm, vias 0 -> 3
- net Standby: track 3.21 -> 121.1 mm, vias 0 -> 3
- net MCLK: track 0.00 -> 104.4 mm, vias 0 -> 4
- net FAULT1: track 3.49 -> 104.2 mm, vias 1 -> 3
- net WARN1: track 2.80 -> 102.8 mm, vias 1 -> 3
- net /Amplifier/AUXADC0: track 0.00 -> 96.4 mm, vias 0 -> 1
- net /Amplifier/SPDIFOUT: track 0.00 -> 90.3 mm, vias 0 -> 1
- net FAULT0: track 3.41 -> 87.4 mm, vias 1 -> 3
- net WARN0: track 2.73 -> 84.8 mm, vias 1 -> 3
- net /Amplifier/SPDIFIN: track 0.00 -> 81.1 mm, vias 0 -> 1
- net +6V: track 27.0 -> 92.5 mm, vias 0 -> 1
- net /Amplifier/SDATAOUT1+: track 0.00 -> 62.3 mm, vias 0 -> 3
- net /Amplifier/SDATAOUT0: track 0.00 -> 62.1 mm, vias 0 -> 3
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
Commit message: Почти все
Parts:
- added REF**: MountingHole_3.2mm_M3, MountingHole:MountingHole_3.2mm_M3, F.Cu at (144.8, 5.08)
- added REF**: MountingHole_3.2mm_M3, MountingHole:MountingHole_3.2mm_M3, F.Cu at (17.8, 43.2)
- added REF**: MountingHole_3.2mm_M3, MountingHole:MountingHole_3.2mm_M3, F.Cu at (54.6, 43.2)
- added REF**: MountingHole_3.2mm_M3, MountingHole:MountingHole_3.2mm_M3, F.Cu at (5.08, 5.08)
- added REF**: MountingHole_3.2mm_M3, MountingHole:MountingHole_3.2mm_M3, F.Cu at (91.4, 43.2)
- added REF**: MountingHole_3.2mm_M3, MountingHole:MountingHole_3.2mm_M3, F.Cu at (144.8, 156.0)
- added REF**: MountingHole_3.2mm_M3, MountingHole:MountingHole_3.2mm_M3, F.Cu at (5.08, 156.0)
- J13: footprint Connector_PinHeader_2.54mm:PinHeader_1x04_P2.54mm_Vertical -> Connector_PinHeader_2.54mm:PinHeader_1x05_P2.54mm_Vertical
- J21, J7: footprint Connector_PinHeader_2.54mm:PinHeader_1x02_P2.54mm_Vertical -> Connector_PinHeader_2.54mm:PinHeader_1x03_P2.54mm_Vertical
- TR1: footprint my:Trans10_Toroid_Horizontal_D60mm -> 00-mylib:Transformer_ETD44_Horizontal
- U15, U16: value MOC3023M -> PC817; footprint Package_DIP:DIP-6_W7.62mm -> Package_DIP:DIP-4_W7.62mm
- moved J16 53.0 mm to (70.6, 86.5)
- moved VD8 36.8 mm to (93.0, 67.3)
- moved VD9 36.8 mm to (129.8, 67.3)
- moved C113 34.8 mm to (84.8, 65.4), turned to 90 degrees
- moved R8 34.6 mm to (56.5, 75.4), turned to 90 degrees
- moved C112 32.0 mm to (124.0, 81.8)
- moved R39 32.0 mm to (126.3, 81.8)
- moved R40 31.4 mm to (121.4, 46.5), turned to 180 degrees
- moved C109 28.1 mm to (105.0, 123.0), turned to 0 degrees
- moved Q1 27.3 mm to (52.8, 75.4), turned to 180 degrees
- moved TR1 26.9 mm to (90.2, 121.6), turned to 0 degrees
- moved C110 26.3 mm to (126.2, 123.1), turned to 0 degrees
- moved R36 24.5 mm to (102.2, 123.0), turned to 180 degrees
- moved C105 24.3 mm to (119.3, 146.0), turned to -90 degrees
- moved R29 23.4 mm to (120.8, 142.2), turned to 0 degrees
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Connections:
- R1 pad 2: Net-(U10-NRST) -> RST
- U10 pad 4: Net-(U10-NRST) -> RST
- U15 pad 3: unconnected-(U15-NC-Pad3) -> Net-(C105-Pad1)
- U15 pad 4: Net-(C105-Pad1) -> Net-(VD14-K)
- U16 pad 3: unconnected-(U16-NC-Pad3) -> Net-(VD15-K)
- U16 pad 4: Net-(VD15-K) -> Net-(C105-Pad1)
- U3 pad 1: Net-(U10-NRST) -> RST
- U6 pad 69: Net-(J13-Pin_1) -> Net-(J13-Pin_4)
- U6 pad 70: Net-(J13-Pin_2) -> Net-(J13-Pin_3)
- U6 pad 71: Net-(J13-Pin_3) -> Net-(J13-Pin_2)
- U6 pad 72: Net-(J13-Pin_4) -> Net-(J13-Pin_1)
- U6 pad 89: (no net) -> GND
Routing:
- net +3V3: track 19.0 -> 443.8 mm, vias 0 -> 16
- net Net-(C105-Pad1): track 2.60 -> 174.8 mm
- net /Amplifier/LRCKOUT1: track 0.00 -> 129.4 mm, vias 0 -> 2
- net /Amplifier/BCLKOUT1: track 0.00 -> 128.1 mm, vias 0 -> 2
- net /Amplifier/SDATAOUT1: track 0.00 -> 127.6 mm, vias 0 -> 2
- net GNDPWR: track 36.5 -> 156.1 mm, vias 0 -> 30
- net /Amplifier/SDATAIN2: track 0.00 -> 115.3 mm, vias 0 -> 3
- net /Amplifier/BCLKIN2: track 0.00 -> 113.7 mm, vias 0 -> 3
- net /Amplifier/LRCKIN2: track 0.00 -> 109.3 mm, vias 0 -> 3
- net REMOTE: track 0.00 -> 109.2 mm, vias 0 -> 2
- net /Amplifier/SDATAOUT3: track 0.00 -> 103.4 mm, vias 0 -> 1
- net /Amplifier/LRCKOUT3: track 0.00 -> 100.1 mm, vias 0 -> 1
- net MCLK: track 104.4 -> 204.1 mm, vias 4 -> 5
- net /Amplifier/BCLKOUT3: track 0.00 -> 99.5 mm, vias 0 -> 1
- net /Amplifier/SDATAIN3: track 0.00 -> 93.3 mm, vias 0 -> 1
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- added copper zone on F.Cu, net +6V
- added copper zone on B.Cu, net GND
- added copper zone on F.Cu, net GND
- added copper zone on B.Cu, net GNDPWR
- added copper zone on F.Cu, net GNDPWR
- added copper zone on B.Cu, net Net-(VD14-A)
- added copper zone on F.Cu, net Net-(VD8-A)
- added copper zone on B.Cu, net Net-(VD8-A1)
- added copper zone on F.Cu, net Net-(VD8-A1)
- added copper zone on B.Cu, net Net-(VD9-A1)
Other:
- board size 149.9 x 171.2 mm -> 149.9 x 160.8 mm

Commit message: Основная плата все
Parts:
- added C16: CAP_10u0_50V_X7R_1206, Capacitor_SMD:C_1206_3216Metric, F.Cu at (97.0, 39.1)
- added R18: 4.7k, Resistor_SMD:R_0603_1608Metric, B.Cu at (104.9, 29.6)
- added R19: 10k, Resistor_SMD:R_0603_1608Metric, F.Cu at (95.2, 22.2)
- added R24: 1k, Resistor_SMD:R_0603_1608Metric, F.Cu at (95.2, 23.9)
- added R42: 1.2k, Resistor_SMD:R_1206_3216Metric, F.Cu at (97.0, 36.7)
- added R43: 4.7k, Resistor_SMD:R_0603_1608Metric, F.Cu at (108.2, 23.5)
- added U5: TLP627, Package_DIP:DIP-4_W7.62mm, F.Cu at (95.6, 33.9)
- C1, C6: value CAP_10u0_25V_X5R_0805 -> CAP_10u0_50V_X7R_1206; footprint Capacitor_SMD:C_0805_2012Metric -> Capacitor_SMD:C_1206_3216Metric
- C102, C111: value 1n -> CAP_1n_50V_X7R_0603; footprint Capacitor_SMD:C_0805_2012Metric -> Capacitor_SMD:C_0603_1608Metric
- C103, C106: value 10n -> CAP_10n_50V_X7R_0603; footprint Capacitor_SMD:C_0805_2012Metric -> Capacitor_SMD:C_0603_1608Metric
- C104: value 2.2μ -> CAP_2u2_50V_X7R_1206
- C105, C125: value 10μ -> CAP_10u0_50V_X7R_1206
- C109, C110: value 22n -> CAP_22n_50V_X7R_0603; footprint Capacitor_SMD:C_0805_2012Metric -> Capacitor_SMD:C_0603_1608Metric
- C112: value 100n -> CAP_100n_50V_X7R_0603; footprint Capacitor_SMD:C_0805_2012Metric -> Capacitor_SMD:C_0603_1608Metric
- C63: footprint Capacitor_SMD:C_0805_2012Metric -> Capacitor_SMD:C_1206_3216Metric
- J12, J19, J20: value Conn_01x06_Male -> Conn_edge_2x6_2.54_Male
- R25, R26, R27, R28, R29, R30, R31, R32, R33, R34, R35, R39: footprint Resistor_SMD:R_0805_2012Metric -> Resistor_SMD:R_0603_1608Metric
- R41: footprint Resistor_SMD:R_0805_2012Metric -> Resistor_SMD:R_1206_3216Metric
- R45: value 330 -> 1k; footprint Resistor_SMD:R_0805_2012Metric -> Resistor_SMD:R_0603_1608Metric
- U15, U16: value PC817 -> TLP627
- VD2: footprint w_smd_diode:do214ac -> Diode_SMD:D_SMA
- moved VD14 19.8 mm to (98.8, 20.4)
- moved VD15 19.8 mm to (102.5, 20.4)
- moved R41 15.4 mm to (101.7, 36.7)
- moved C125 15.3 mm to (101.7, 39.1)
- moved R45 13.2 mm to (106.4, 37.1)
- moved U16 8.02 mm to (107.4, 33.9), turned to 90 degrees
- moved U15 7.60 mm to (101.6, 33.9), turned to 90 degrees
- moved L18 2.29 mm to (140.2, 23.0)
- moved C2 1.40 mm to (38.5, 39.6)
- moved U7 0.88 mm to (80.0, 138.3)
- moved VD2 0.81 mm to (35.4, 39.4)
- moved C6 0.80 mm to (35.4, 79.5)
- moved C60 0.76 mm to (80.1, 135.4)
- moved C50 0.68 mm to (33.4, 78.9)
- moved C1 0.63 mm to (43.2, 76.7)
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Connections:
- C105 pad 1: Net-(C105-Pad1) -> Net-(VD14-K)
- C107 pad 1: Net-(VD14-A) -> Net-(C107-Pad1)
- C108 pad 1: Net-(VD14-A) -> Net-(C107-Pad1)
- C109 pad 2: Net-(VD14-A) -> Net-(C107-Pad1)
- C110 pad 1: Net-(VD14-A) -> Net-(C107-Pad1)
- L18 pad 2: Net-(VD14-A) -> Net-(C107-Pad1)
- R29 pad 1: Net-(C105-Pad1) -> Net-(VD14-K)
- TR1 pad 2: Net-(VD14-A) -> Net-(C107-Pad1)
- TR1 pad 3: Net-(VD14-A) -> Net-(C107-Pad1)
- U10 pad 10: REMOTE -> unconnected-(U10-PA4-Pad10)
- U12 pad 12: unconnected-(U12-GPIO_A6-Pad12) -> ACC_IN
- U12 pad 7: unconnected-(U12-GPIO_G11-Pad7) -> REMOTE
- U15 pad 3: Net-(C105-Pad1) -> Net-(VD14-A)
- U15 pad 4: Net-(VD14-K) -> Net-(C107-Pad1)
- U16 pad 3: Net-(VD15-K) -> Net-(VD15-A)
- U16 pad 4: Net-(C105-Pad1) -> Net-(C107-Pad1)
- VD15 pad 1: Net-(VD15-K) -> Net-(VD14-K)
- VD15 pad 2: Net-(VD14-A) -> Net-(VD15-A)
Routing:
- net Net-(VD14-K): track 10.4 -> 187.7 mm, vias 0 -> 2
- net Net-(C105-Pad1): track 174.8 -> 0.00 mm
- net ACC_IN: track 0.00 -> 129.7 mm, vias 0 -> 2
- net Net-(VD14-A): track 80.7 -> 10.3 mm, vias 1 -> 0
- net Net-(C107-Pad1): track 0.00 -> 68.3 mm
- net +6V: track 7.46 -> 65.9 mm, vias 1 -> 2
- net REMOTE: track 109.2 -> 149.6 mm, vias 2 -> 3
- net +3V3: track 443.8 -> 471.6 mm, vias 16 -> 18
- net ACC: track 19.8 -> 39.2 mm
- net GNDPWR: track 156.1 -> 172.0 mm
- net Net-(VD15-K): track 9.81 -> 0.00 mm
- net Net-(VD15-A): track 0.00 -> 9.21 mm
- net Net-(C16-Pad1): track 0.00 -> 5.51 mm
- net Net-(R19-Pad1): track 0.00 -> 4.92 mm
- net Net-(VD1-K): track 4.41 -> 6.75 mm
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- added copper zone on B.Cu, net Net-(C107-Pad1)
- added copper zone on B.Cu, net Net-(VD10-A)
- removed copper zone on B.Cu, net Net-(VD14-A)
- removed copper zone on B.Cu, net Net-(VD9-A1)

Commit message: Добавил надписи
Parts:
- moved J10 2.54 mm to (84.6, 71.9)
Other:
- board text added: "+"
- board text added: "+6V"
- board text added: "ADC in"
- board text added: "GND"
- board text added: "I2S In"
- board text added: "I2S Out"
- board text added: "In"
- board text added: "MP14"
- board text added: "MP15"
- board text added: "MP16"
- board text added: "MP17"
- board text added: "MP18"
- board text added: "MP19"
- board text added: "MP20"
- board text added: "MP21"
- board text added: "RX"
- board text added: "SPDIF"
- board text added: "SWBCLK"
- board text added: "SWBDIO"
- board text added: "TX"
- board text added: "UART"

Commit message: Почти все
Parts:
- L19: footprint my:L_Axial_L26.0mm_D9.0mm_P5.08mm_Vertical -> 00-mylib:L_Toroid_Vertical_L33.0mm_W17.8mm_P12.70mm_Pulse_KM-5
- moved R40 15.2 mm to (136.6, 46.2)
- moved C115 12.1 mm to (122.2, 44.5)
- moved L19 11.0 mm to (114.0, 62.9), turned to 180 degrees
- moved C114 9.04 mm to (111.6, 44.4), turned to 90 degrees
- moved C74 6.28 mm to (64.0, 33.7), turned to 90 degrees
- moved C73 5.47 mm to (64.4, 34.7), turned to -90 degrees
- moved C108 4.75 mm to (142.5, 38.4)
- moved C64 3.98 mm to (83.6, 45.5), turned to 0 degrees
- moved REF** 3.06 mm to (145.0, 152.9)
- moved REF** 3.06 mm to (5.33, 152.9)
- moved C47 0.46 mm to (45.9, 44.9)
Routing:
- net +3V3: track 471.6 -> 485.1 mm, vias 18 -> 22
- net ACC_IN: track 129.7 -> 137.2 mm, vias 2 -> 9
- net PVDD: track 9.81 -> 16.2 mm
- net Net-(VD9-A1): track 40.9 -> 45.7 mm
- net REMOTE: track 149.6 -> 153.4 mm, vias 3 -> 5
- net Net-(VD14-K): track 187.7 -> 190.8 mm, vias 2 -> 6
- net VBAT: track 70.0 -> 68.8 mm
- net /Amplifier/SDATAOUT2: track 18.7 -> 19.3 mm
- net GNDPWR: vias 30 -> 32
- net GND: vias 64 -> 78
- added copper zone on B.Cu, net Net-(VD9-A1)
- removed copper zone on B.Cu, net Net-(VD10-A)
Other:
- board size 149.9 x 160.8 mm -> 149.9 x 157.7 mm

Commit message: Добавил корпус
Parts:
- moved F1 2.03 mm to (134.6, 11.6)
- moved VD1 1.90 mm to (130.8, 19.6)
- moved REF** 0.36 mm to (5.08, 152.7)
- moved REF** 0.36 mm to (144.8, 152.7)
Changed lines of the file:
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@@
 	(footprint "00-mylib:Fuse_Blade_vertical"
 		(layer "F.Cu")
-		(at 134.66 9.525 90)
+		(at 134.62 11.555 90)
 		(descr "car blade fuse direct solder")
 		(tags "car blade fuse")
@@
 	(footprint "Diode_SMD:D_SMC"
 		(layer "F.Cu")
-		(at 130.146 17.78 180)
+		(at 130.81 19.558 180)
 		(descr "Diode SMC (DO-214AB)")
 		(tags "Diode SMC (DO-214AB)")
@@
 			(at 0 -4.2 0)
 			(layer "F.SilkS")
+			(hide yes)
 			(effects
 				(font
@@
 			(at 0 0 0)
 			(layer "F.Fab")
+			(hide yes)
 			(effects
 				(font
@@
 			(at 0 -4.2 0)
 			(layer "F.SilkS")
+			(hide yes)
 			(effects
 				(font
@@
 			(at 0 0 0)
 			(layer "F.Fab")
+			(hide yes)
 			(effects
 				(font
@@
 			(at 0 -4.2 0)
 			(layer "F.SilkS")
+			(hide yes)
 			(effects
 				(font
@@
 			(at 0 0 0)
 			(layer "F.Fab")
+			(hide yes)
 			(effects
 				(font
@@
 		(locked yes)
 		(layer "F.Cu")
-		(at 145.034 152.908)
+		(at 144.78 152.654)
 		(descr "Mounting Hole 3.2mm, no annular, M3")
 		(tags "mounting hole 3.2mm no annular m3")
@@
 		(locked yes)
 		(layer "F.Cu")
-		(at 5.334 152.908)
+		(at 5.08 152.654)
 		(descr "Mounting Hole 3.2mm, no annular, M3")
 		(tags "mounting hole 3.2mm no annular m3")
@@
 	)
 	(segment
+		(start 127.41 19.558)
+		(end 124.968 19.558)
+		(width 4)
+		(layer "F.Cu")
+		(net 76)
+	)
+	(segment
 		(start 111.8895 145.4175)
 		(end 111.9305 145.4175)
@@
 	)
 	(segment
-		(start 126.746 17.78)
-		(end 119.852729 24.673271)
+		(start 119.852729 24.673271)
+		(end 119.852729 27.94)
 		(width 4)
 		(layer "F.Cu")
@@
 	)
 	(segment
-		(start 119.852729 24.673271)
-		(end 119.852729 27.94)
+		(start 124.968 19.558)
+		(end 119.852729 24.673271)
 		(width 4)
 		(layer "F.Cu")
@@
 	)
 	(segment
-		(start 140.208 17.987)
-		(end 140.081 17.86)
+		(start 134.308 19.558)
+		(end 134.21 19.558)
+		(width 4)
+		(layer "F.Cu")
+		(net 231)
+	)
+	(segment
+		(start 136.006 17.86)
+		(end 134.308 19.558)
 		(width 4)
 		(layer "F.Cu")
@@
 	(segment
 		(start 140.081 17.86)
-		(end 133.626 17.86)
+		(end 136.006 17.86)
 		(width 4)
 		(layer "F.Cu")
@@
 	)
 	(segment
-		(start 133.626 17.86)
-		(end 133.546 17.78)
+		(start 140.208 17.987)
+		(end 140.081 17.86)
 		(width 4)
 		(layer "F.Cu")
