File: daw00/spdif/spdif.kicad_pcb (KiCad board)
At the start: 2 copper layers, 25.4 x 31.7 mm, 8 parts, among them J1 Conn_01x06_Male, U1 DLR1160, U2 DLR1160

Commit message: Почти все
Parts:
- added REF**: MountingHole_3.2mm_M3, MountingHole:MountingHole_3.2mm_M3, F.Cu at (99.1, 64.8)
Other:
- board size 25.4 x 31.7 mm -> 25.4 x 40.6 mm

Commit message: Добавил корпус
Parts:
- moved U1 4.68 mm to (96.5, 51.8)
- moved U2 4.68 mm to (96.5, 41.1)
Routing:
- net Net-(U1-VCC): track 12.4 -> 17.8 mm
- net Net-(U2-VIN): track 12.2 -> 17.6 mm
- net /SPDIFOUT: track 31.3 -> 36.1 mm
- net /SPDIFIN: track 14.1 -> 13.1 mm
Changed lines of the file:
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@@
 	(footprint "my:Toslink"
 		(layer "F.Cu")
-		(at 92.964 38.1 -90)
+		(at 96.52 41.148 -90)
 		(property "Reference" "U2"
 			(at 0 -9.652 90)
@@
 	(footprint "my:Toslink"
 		(layer "F.Cu")
-		(at 92.964 48.768 -90)
+		(at 96.52 51.816 -90)
 		(property "Reference" "U1"
 			(at 0 -9.652 90)
@@
 	)
 	(segment
+		(start 93.89 48.26)
+		(end 93.89 49.276)
+		(width 0.625)
+		(layer "B.Cu")
+		(net 2)
+	)
+	(segment
 		(start 83.095 48.831)
 		(end 83.794 49.53)
@@
 	(segment
 		(start 83.095 45.974)
+		(end 83.095 48.831)
+		(width 0.625)
+		(layer "B.Cu")
+		(net 2)
+	)
+	(segment
+		(start 83.095 45.974)
 		(end 84.5575 44.5115)
 		(width 0.625)
@@
 	)
 	(segment
-		(start 88.6175 44.5115)
-		(end 90.334 46.228)
+		(start 84.5575 44.5115)
+		(end 90.1415 44.5115)
 		(width 0.625)
 		(layer "B.Cu")
@@
 	)
 	(segment
-		(start 83.095 45.974)
-		(end 83.095 48.831)
-		(width 0.625)
-		(layer "B.Cu")
-		(net 2)
-	)
-	(segment
-		(start 84.5575 44.5115)
-		(end 88.6175 44.5115)
+		(start 90.1415 44.5115)
+		(end 93.89 48.26)
 		(width 0.625)
 		(layer "B.Cu")
@@
 	)
 	(segment
+		(start 84.7235 33.8435)
+		(end 90.1415 33.8435)
+		(width 0.625)
+		(layer "B.Cu")
+		(net 3)
+	)
+	(segment
+		(start 90.1415 33.8435)
+		(end 93.89 37.592)
+		(width 0.625)
+		(layer "B.Cu")
+		(net 3)
+	)
+	(segment
 		(start 83.261 35.306)
 		(end 84.7235 33.8435)
@@
 	)
 	(segment
-		(start 88.6175 33.8435)
-		(end 90.334 35.56)
-		(width 0.625)
-		(layer "B.Cu")
-		(net 3)
-	)
-	(segment
-		(start 84.7235 33.8435)
-		(end 88.6175 33.8435)
-		(width 0.625)
-		(layer "B.Cu")
-		(net 3)
-	)
-	(segment
 		(start 83.261 38.329)
 		(end 83.794 38.862)
@@
 	)
 	(segment
-		(start 88.9 52.742)
-		(end 90.334 51.308)
+		(start 93.89 37.592)
+		(end 93.89 38.608)
+		(width 0.625)
+		(layer "B.Cu")
+		(net 3)
+	)
+	(segment
+		(start 88.9 64.77)
+		(end 88.9 58.33)
 		(width 1.27)
 		(layer "B.Cu")
@@
 	)
 	(segment
-		(start 88.9 64.77)
-		(end 88.9 52.742)
+		(start 92.874 54.356)
+		(end 93.89 54.356)
 		(width 1.27)
 		(layer "B.Cu")
 		(net 5)
+	)
+	(segment
+		(start 88.9 58.33)
+		(end 92.874 54.356)
+		(width 1.27)
+		(layer "B.Cu")
+		(net 5)
+	)
+	(segment
+		(start 81.735 49.4513)
+		(end 81.735 44.503)
+		(width 1.27)
+		(layer "B.Cu")
+		(net 8)
+	)
+	(segment
+		(start 90.842 40.64)
+		(end 93.89 43.688)
+		(width 1.27)
+		(layer "B.Cu")
+		(net 8)
 	)
 	(segment
@@
 	)
 	(segment
-		(start 81.735 49.4513)
-		(end 81.735 44.503)
-		(width 1.27)
-		(layer "B.Cu")
-		(net 8)
-	)
-	(segment
 		(start 83.82 51.5363)
 		(end 81.735 49.4513)
@@
 	(segment
 		(start 85.598 40.64)
-		(end 90.334 40.64)
+		(end 90.842 40.64)
 		(width 1.27)
 		(layer "B.Cu")
